Commit message: 更新机器人描述和控制配置，修正关节位置限制，添加初始化角度发布节点，重命名动画显示启动文件

File: src/robot_description/urdf/robot_description.xacro (robot description, xacro)
@@ -83,5 +83,5 @@
     <child link="dummy_point3"/>
     <!-- 如果需要在 truss_link 坐标系中给 base_link 设置一个平移或姿态偏移，可以在这里修改 xyz / rpy -->
-    <origin xyz="0.1325 0.13 0.1325" rpy="1.5708 0 0"/>
+    <origin xyz="0.1325 0.23 0.35" rpy="1.5708 0 0"/>
   </joint>
   <link name="dummy_point3"></link>
@@ -91,5 +91,5 @@
     <!-- 如果需要在 truss_link 坐标系中给 base_link 设置一个平移或姿态偏移，可以在这里修改 xyz / rpy -->
     <!-- 转换到joint2_6______0.1 -->
-    <origin xyz="0 0.115 -0.3" rpy="0 0 0"/>
+    <origin xyz="0 0.215 -0.3" rpy="0 0 0"/>
   </joint>
   <link name="dummy_point4"></link>

Commit message: 添加新的文件和功能以支持机器人控制和姿态计算，包括笛卡尔插值服务和机器人姿态服务，更新相关配置文件，修正变换矩阵的加载逻辑，增强文档和代码的清晰度。

File: src/robot_description/urdf/robot_description.xacro (robot description, xacro)
@@ -94,4 +94,12 @@
   </joint>
   <link name="dummy_point4"></link>
+  <joint name="truss_link_to_obj" type="fixed">
+    <parent link="truss_link"/>
+    <child link="object"/>
+    <!-- 如果需要在 truss_link 坐标系中给 base_link 设置一个平移或姿态偏移，可以在这里修改 xyz / rpy -->
+    <!-- 转换到joint2_6______0.1 -->
+    <origin xyz="0.1325 0.13 0.35" rpy="0 0 0"/>
+  </joint>
+  <link name="object"></link>
   <link name="base_link">
     <inertial>

Commit message: temp

File: src/robot_description/urdf/robot_description.xacro (robot description, xacro)
@@ -99,5 +99,5 @@
     <!-- 如果需要在 truss_link 坐标系中给 base_link 设置一个平移或姿态偏移，可以在这里修改 xyz / rpy -->
     <!-- 转换到joint2_6______0.1 -->
-    <origin xyz="0.1325 0.13 0.35" rpy="0 0 0"/>
+    <origin xyz="0.1325 0.03 0.35" rpy="1.5708 0 0"/>
   </joint>
   <link name="object"></link>

Commit message: temp

File: src/robot_description/urdf/robot_description.xacro (robot description, xacro)
@@ -102,4 +102,12 @@
   </joint>
   <link name="object"></link>
+  <joint name="truss_link_to_obj1" type="fixed">
+    <parent link="truss_link"/>
+    <child link="object1"/>
+    <!-- 如果需要在 truss_link 坐标系中给 base_link 设置一个平移或姿态偏移，可以在这里修改 xyz / rpy -->
+    <!-- 转换到joint2_6______0.1 -->
+    <origin xyz="0 0.215 0.3" rpy="0 3.1416 0"/>
+  </joint>
+  <link name="object1"></link>
   <link name="base_link">
     <inertial>

Commit message: 完成基本动作

File: src/robot_description/urdf/robot_description.xacro (robot description, xacro)
@@ -83,5 +83,5 @@
     <child link="dummy_point3"/>
     <!-- 如果需要在 truss_link 坐标系中给 base_link 设置一个平移或姿态偏移，可以在这里修改 xyz / rpy -->
-    <origin xyz="0.1325 0.23 0.35" rpy="1.5708 0 0"/>
+    <origin xyz="0.1325 0.23 0.35" rpy="1.5708 1.5708 0"/>
   </joint>
   <link name="dummy_point3"></link>
@@ -99,5 +99,5 @@
     <!-- 如果需要在 truss_link 坐标系中给 base_link 设置一个平移或姿态偏移，可以在这里修改 xyz / rpy -->
     <!-- 转换到joint2_6______0.1 -->
-    <origin xyz="0.1325 0.03 0.35" rpy="1.5708 0 0"/>
+    <origin xyz="0.1325 0.03 0.35" rpy="1.5708 1.5708 0"/>
   </joint>
   <link name="object"></link>
@@ -107,7 +107,15 @@
     <!-- 如果需要在 truss_link 坐标系中给 base_link 设置一个平移或姿态偏移，可以在这里修改 xyz / rpy -->
     <!-- 转换到joint2_6______0.1 -->
-    <origin xyz="0 0.215 0.3" rpy="0 3.1416 0"/>
+    <origin xyz="-0.1 0.215 0.085" rpy="0 3.1416 0"/>
   </joint>
   <link name="object1"></link>
+  <joint name="truss_link_to_obj2" type="fixed">
+    <parent link="truss_link"/>
+    <child link="object2"/>
+    <!-- 如果需要在 truss_link 坐标系中给 base_link 设置一个平移或姿态偏移，可以在这里修改 xyz / rpy -->
+    <!-- 转换到joint2_6______0.1 -->
+    <origin xyz="-0.265 0.215 -0.35" rpy="0 0 -1.5708"/>
+  </joint>
+  <link name="object2"></link>
   <link name="base_link">
     <inertial>

Commit message: temp 需要更改初始关节角

File: src/robot_description/urdf/robot_description.xacro (robot description, xacro)
@@ -83,5 +83,5 @@
     <child link="dummy_point3"/>
     <!-- 如果需要在 truss_link 坐标系中给 base_link 设置一个平移或姿态偏移，可以在这里修改 xyz / rpy -->
-    <origin xyz="0.1325 0.23 0.35" rpy="1.5708 1.5708 0"/>
+    <origin xyz="0.1325 0.06 0.35" rpy="1.5708 1.5708 0"/>
   </joint>
   <link name="dummy_point3"></link>

Commit message: 修改单臂操作

File: src/robot_description/urdf/robot_description.xacro (robot description, xacro)
@@ -83,5 +83,5 @@
     <child link="dummy_point3"/>
     <!-- 如果需要在 truss_link 坐标系中给 base_link 设置一个平移或姿态偏移，可以在这里修改 xyz / rpy -->
-    <origin xyz="0.1325 0.06 0.35" rpy="1.5708 1.5708 0"/>
+    <origin xyz="0.08 0.18 0.40" rpy="1.5708 0.707 0"/>
   </joint>
   <link name="dummy_point3"></link>
@@ -99,5 +99,5 @@
     <!-- 如果需要在 truss_link 坐标系中给 base_link 设置一个平移或姿态偏移，可以在这里修改 xyz / rpy -->
     <!-- 转换到joint2_6______0.1 -->
-    <origin xyz="0.1325 0.03 0.35" rpy="1.5708 1.5708 0"/>
+    <origin xyz="0.08 0.03 0.40" rpy="1.5708 0.707 0"/>
   </joint>
   <link name="object"></link>

Commit message: temp

File: src/robot_description/urdf/robot_description.xacro (robot description, xacro)
@@ -118,4 +118,20 @@
   </joint>
   <link name="object2"></link>
+  <link name="cube_l"></link>
+  <joint name="truss_link_to_cube_l" type="fixed">
+    <parent link="truss_link"/>
+    <child link="cube_l"/>
+    <!-- 如果需要在 truss_link 坐标系中给 base_link 设置一个平移或姿态偏移，可以在这里修改 xyz / rpy -->
+    <!-- 转换到joint2_6______0.1 -->
+    <origin xyz="-0.1175 0.12 0.2325" rpy="0 3.1416 0"/>
+  </joint>
+  <link name="cube_r"></link>
+  <joint name="truss_link_to_cube_r" type="fixed">
+    <parent link="truss_link"/>
+    <child link="cube_r"/>
+    <!-- 如果需要在 truss_link 坐标系中给 base_link 设置一个平移或姿态偏移，可以在这里修改 xyz / rpy -->
+    <!-- 转换到joint2_6______0.1 -->
+    <origin xyz="-0.1175 0.12 -0.2325" rpy="0 0 0"/>
+  </joint>
   <link name="base_link">
     <inertial>
