Commit message: temp

File: src/robot_description/urdf/robot_description copy.xacro (robot description, xacro)
@@ -5,5 +5,5 @@
 <robot name="robot_description"  xmlns:xacro="http://ros.org/wiki/xacro">
   <xacro:arg name="transmission_hw_interface" default = "hardware_interface/EffortJointInterface"/>
-  <xacro:include filename = "$(find robotiq_2f_85_gripper_visualization)/urdf/robotiq_arg2f_85_macro.xacro"/>
+  <xacro:include filename = "$(find robotiq_2f_85_gripper_gazebo)/urdf/robotiq_arg2f_85_macro.xacro"/>
   <xacro:include filename="robot_parameter.xacro" />
 <!--body*********************************************************************************************************-->
@@ -11,6 +11,126 @@
   <joint name="world_joint" type="fixed">
     <parent link="world"/>
-    <child  link="base_link"/>
+    <child  link="dummy_link"/>
     <origin xyz="0 0 0.45" rpy="0 1.5708 0"/>
+  </joint>
+  <link name="dummy_link"></link>
+  <joint name="dummy_joint" type="fixed">
+      <parent link="dummy_link"/>
+      <child  link="base_link"/>
+      <origin xyz="0 0 0" rpy="0 0 0"/>
+  </joint>
+  <joint name="world_to_truss_link" type="fixed">
+    <parent link="world"/>
+    <child link="truss_link"/>
+    <!-- 如果需要在世界坐标系中给 truss_link 设置一个平移或姿态偏移，可以在这里修改 xyz / rpy -->
+    <origin xyz="0.6625 0 0" rpy="1.5708 0 3.1415"/>
+  </joint>
+  <link name="truss_link">
+    <inertial>
+      <origin
+        xyz="0.36747875296263 -0.0267703008644749 2.17639122268576E-06"
+        rpy="0 0 0" />
+      <mass
+        value="21.7746312239973" />
+      <inertia
+        ixx="6.13854571738268"
+        ixy="0.0126716758688149"
+        ixz="-0.000126373819517297"
+        iyy="16.7375552194284"
+        iyz="-1.43555608026521E-06"
+        izz="10.6624119014708" />
+    </inertial>
+    <visual>
+      <origin
+        xyz="0 0 0"
+        rpy="0 0 0" />
+      <geometry>
+        <mesh
+          filename="package://robot_description/meshes/truss_link.STL" />
+      </geometry>
+      <material
+        name="">
+        <color
+          rgba="0.792156862745098 0.819607843137255 0.933333333333333 1" />
+      </material>
+    </visual>
+    <collision>
+      <origin
+        xyz="0 0 0"
+        rpy="0 0 0" />
+      <geometry>
+        <mesh
+          filename="package://robot_description/meshes/truss_link.STL" />
+      </geometry>
+    </collision>
+  </link>
+  <joint name="truss_link_to_point1" type="fixed">
+    <parent link="truss_link"/>
+    <child link="dummy_point1"/>
+    <!-- 如果需要在 truss_link 坐标系中给 base_link 设置一个平移或姿态偏移，可以在这里修改 xyz / rpy -->
+    <origin xyz="0.795 0 0.53" rpy="1.5708 0 0"/>
+  </joint>
+  <link name="dummy_point1"></link>
+  <joint name="truss_link_to_point2" type="fixed">
+    <parent link="truss_link"/>
+    <child link="dummy_point2"/>
+    <!-- 如果需要在 truss_link 坐标系中给 base_link 设置一个平移或姿态偏移，可以在这里修改 xyz / rpy -->
+    <origin xyz="0.795 0 -0.53" rpy="1.5708 0 0"/>
+  </joint>
+  <link name="dummy_point2"></link>
+  <joint name="truss_link_to_point3" type="fixed">
+    <parent link="truss_link"/>
+    <child link="dummy_point3"/>
+    <!-- 如果需要在 truss_link 坐标系中给 base_link 设置一个平移或姿态偏移，可以在这里修改 xyz / rpy -->
+    <origin xyz="0.08 0.18 0.40" rpy="1.5708 0.707 0"/>
+  </joint>
+  <link name="dummy_point3"></link>
+  <joint name="truss_link_to_point4" type="fixed">
+    <parent link="truss_link"/>
+    <child link="dummy_point4"/>
+    <!-- 如果需要在 truss_link 坐标系中给 base_link 设置一个平移或姿态偏移，可以在这里修改 xyz / rpy -->
+    <!-- 转换到joint2_6______0.1 -->
+    <origin xyz="0 0.215 -0.3" rpy="0 0 0"/>
+  </joint>
+  <link name="dummy_point4"></link>
+  <joint name="truss_link_to_obj" type="fixed">
+    <parent link="truss_link"/>
+    <child link="object"/>
+    <!-- 如果需要在 truss_link 坐标系中给 base_link 设置一个平移或姿态偏移，可以在这里修改 xyz / rpy -->
+    <!-- 转换到joint2_6______0.1 -->
+    <origin xyz="0.08 0.03 0.40" rpy="1.5708 0.707 0"/>
+  </joint>
+  <link name="object"></link>
+  <joint name="truss_link_to_obj1" type="fixed">
+    <parent link="truss_link"/>
+    <child link="object1"/>
+    <!-- 如果需要在 truss_link 坐标系中给 base_link 设置一个平移或姿态偏移，可以在这里修改 xyz / rpy -->
+    <!-- 转换到joint2_6______0.1 -->
+    <origin xyz="-0.1 0.215 0.085" rpy="0 3.1416 0"/>
+  </joint>
+  <link name="object1"></link>
+  <joint name="truss_link_to_obj2" type="fixed">
+    <parent link="truss_link"/>
+    <child link="object2"/>
+    <!-- 如果需要在 truss_link 坐标系中给 base_link 设置一个平移或姿态偏移，可以在这里修改 xyz / rpy -->
+    <!-- 转换到joint2_6______0.1 -->
+    <origin xyz="-0.265 0.215 -0.35" rpy="0 0 -1.5708"/>
+  </joint>
+  <link name="object2"></link>
+  <link name="cube_l"></link>
+  <joint name="truss_link_to_cube_l" type="fixed">
+    <parent link="truss_link"/>
+    <child link="cube_l"/>
+    <!-- 如果需要在 truss_link 坐标系中给 base_link 设置一个平移或姿态偏移，可以在这里修改 xyz / rpy -->
+    <!-- 转换到joint2_6______0.1 -->
+    <origin xyz="-0.1175 0.12 0.2325" rpy="0 3.1416 0"/>
+  </joint>
+  <link name="cube_r"></link>
+  <joint name="truss_link_to_cube_r" type="fixed">
+    <parent link="truss_link"/>
+    <child link="cube_r"/>
+    <!-- 如果需要在 truss_link 坐标系中给 base_link 设置一个平移或姿态偏移，可以在这里修改 xyz / rpy -->
+    <!-- 转换到joint2_6______0.1 -->
+    <origin xyz="-0.1175 0.12 -0.2325" rpy="0 0 0"/>
   </joint>
   <link name="base_link">
@@ -20,5 +140,7 @@
       <inertia ixx="0.004886486" ixy="-0.000017397" ixz="-0.000263075" iyy="0.004100237" iyz="0" izz="0.003937989" />
     </inertial>
-    <visual>
+<!--重心:(毫米)	X = -0.880	Y = -0.663	Z = 42.409
+    惯性张量: (千克*平方毫米)由重心决定，并且对齐输出的坐标系。Lxx = 4886.486 Lxy = -17.397 Lxz = -263.075 Lyy = 4100.238 Lyz = 0.709 Lzz = 3937.989-->
+     <visual>
       <origin xyz="0 0 0" rpy="0 0 0" />
       <geometry> <mesh filename="package://robot_description/meshes/base_link.STL" /> </geometry>
@@ -26,8 +148,7 @@
     </visual>
     <collision>
-      <origin xyz="0 0 0" rpy="0 0 0" />
-      <geometry>
-        <mesh filename="package://robot_description/meshes/base_link.STL"/>
-      </geometry>
+      <origin xyz="0 0 0.04" rpy="0 0 0" />
+      <geometry> <box size="0.10 0.10 0.14" /> </geometry>
+      <!--geometry> <mesh filename="package://robot_description/meshes/base_link.STL" /> </geometry-->
       <surface>
         <friction>
@@ -41,90 +162,4 @@
     </collision>
   </link>
-  <joint name="world_to_truss_link" type="fixed">
-    <parent link="world"/>
-    <child link="truss_link"/>
-    <origin xyz="0.6625 0 0" rpy="1.5708 0 3.1415"/>
-  </joint>
-  <link name="truss_link">
-    <inertial>
-      <origin xyz="0.36747875296263 -0.0267703008644749 2.17639122268576E-06" rpy="0 0 0" />
-      <mass value="21.7746312239973" />
-      <inertia ixx="6.13854571738268" ixy="0.0126716758688149" ixz="-0.000126373819517297"
-               iyy="16.7375552194284" iyz="-1.43555608026521E-06" izz="10.6624119014708" />
-    </inertial>
-    <visual>
-      <origin xyz="0 0 0" rpy="0 0 0" />
-      <geometry>
-        <mesh
-          filename="package://robot_description/meshes/truss_link.STL" />
-      </geometry>
-      <material
-        name="">
-        <color
-          rgba="0.792156862745098 0.819607843137255 0.933333333333333 1" />
-      </material>
-    </visual>
-    <collision>
-      <origin xyz="0 0 0" rpy="0 0 0" />
-      <geometry>
-        <mesh
-          filename="package://robot_description/meshes/truss_link.STL" />
-      </geometry>
-    </collision>
-  </link>
-  <!-- <link name="dummy_point1"></link>
-  <joint name="truss_link_to_point1" type="fixed">
-    <parent link="truss_link"/>
-    <child link="dummy_point1"/>
-    <origin xyz="0.795 0 0.53" rpy="1.5708 0 0"/>
-  </joint>
-  <link name="dummy_point2"></link>
-  <joint name="truss_link_to_point2" type="fixed">
-    <parent link="truss_link"/>
-    <child link="dummy_point2"/>
-    <origin xyz="0.795 0 -0.53" rpy="1.5708 0 0"/>
-  </joint>
-  <link name="dummy_point3"></link>
-  <joint name="truss_link_to_point3" type="fixed">
-    <parent link="truss_link"/>
-    <child link="dummy_point3"/>
-    <origin xyz="0.08 0.18 0.40" rpy="1.5708 0.707 0"/>
-  </joint>
-  <link name="dummy_point4"></link>
-  <joint name="truss_link_to_point4" type="fixed">
-    <parent link="truss_link"/>
-    <child link="dummy_point4"/>
-    <origin xyz="0 0.215 -0.3" rpy="0 0 0"/>
-  </joint>
-  <link name="object"></link>
-  <joint name="truss_link_to_obj" type="fixed">
-    <parent link="truss_link"/>
-    <child link="object"/>
-    <origin xyz="0.08 0.03 0.40" rpy="1.5708 0.707 0"/>
-  </joint>
-  <link name="object1"></link>
-  <joint name="truss_link_to_obj1" type="fixed">
-    <parent link="truss_link"/>
-    <child link="object1"/>
-    <origin xyz="-0.1 0.215 0.085" rpy="0 3.1416 0"/>
-  </joint>
-  <link name="object2"></link>
-  <joint name="truss_link_to_obj2" type="fixed">
-    <parent link="truss_link"/>
-    <child link="object2"/>
-    <origin xyz="-0.265 0.215 -0.35" rpy="0 0 -1.5708"/>
-  </joint>
-  <link name="cube_l"></link>
-  <joint name="truss_link_to_cube_l" type="fixed">
-    <parent link="truss_link"/>
-    <child link="cube_l"/>
-    <origin xyz="-0.1175 0.12 0.2325" rpy="0 3.1416 0"/>
-  </joint>
-  <link name="cube_r"></link>
-  <joint name="truss_link_to_cube_r" type="fixed">
-    <parent link="truss_link"/>
-    <child link="cube_r"/>
-    <origin xyz="-0.1175 0.12 -0.2325" rpy="0 0 0"/>
-  </joint> -->
   <link name="Link_platform">
     <inertial>
@@ -133,4 +168,6 @@
       <inertia ixx="0.000745872" ixy="0" ixz="0" iyy="0.000792081" iyz="0" izz="0.001494320" />
     </inertial>
+<!--重心:(毫米)	X = 0.000	Y = 0.000	Z = 11.605
+    惯性张量: (千克* 平方毫米)由重心决定，并且对齐输出的坐标系。Lxx = 745.872	Lxy = 0.000	Lxz = 0.000	Lyy = 792.081	Lyz = 0.000	Lzz = 1494.320-->
     <visual>
       <origin xyz="0 0 0" rpy="0 0 0" />
@@ -138,8 +175,8 @@
       <material name=""> <color rgba="0.75294 0.75294 0.75294 1" /> </material>
     </visual>
-    <collision>
+    <!--collision>
       <origin xyz="0 0 0" rpy="0 0 0" />
       <geometry> <mesh filename="package://robot_description/meshes/Link_platform.STL" /> </geometry>
-    </collision>
+    </collision-->
   </link>
   <joint name="Joint_platform" type="prismatic">
@@ -149,5 +186,9 @@
     <axis xyz="0 0 1" />
     <xacro:insert_block name="negative_dynamics_parameter"/>
-    <limit lower="0" upper="0.5" effort="1000" velocity="10" />
+    <limit
+      lower="0"
+      upper="0.5"
+      effort="1000"
+      velocity="10" />
   </joint>
 <!--leg*********************************************************************************************************-->
@@ -159,4 +200,6 @@
       <inertia ixx="0.000648473" ixy="-0.001018876" ixz="0.000012959" iyy="0.002674366" iyz="0" izz="0.003031056" />
     </inertial>
+<!--重心:(毫米)	X = 85.427 Y = -25.518 Z = -0.131
+    惯性张量: (千克*平方毫米)由重心决定，并且对齐输出的坐标系。Lxx = 648.473	Lxy = -1018.876	Lxz = 12.959 Lyy = 2674.366	Lyz = 0.781	Lzz = 3031.056-->
     <visual>
       <origin xyz="0 0 0" rpy="0 0 0" />
@@ -164,8 +207,8 @@
       <material name=""> <color rgba="0 1 1 1" /> </material>
     </visual>
-    <collision>
+    <!--collision>
       <origin xyz="0 0 0" rpy="0 0 0" />
       <geometry> <mesh filename="package://robot_description/meshes/Link_0.STL" /> </geometry>
-    </collision>
+    </collision-->
   </link>
   <joint name="Joint${number}_0" type="revolute">
@@ -187,4 +230,6 @@
       <inertia ixx="0.000671687" ixy="-0.000084224" ixz="-0.000107815" iyy="0.000786758" iyz="0.000017298" izz="0.000958254" />
     </inertial>
+<!--重心:(毫米)	X = 52.469 Y = -9.040	Z = 2.060
+    惯性张量:(千克*平方毫米)由重心决定，并且对齐输出的坐标系。Lxx = 671.687	Lxy = -84.224	Lxz = -107.815 Lyy = 786.758 Lyz = 17.298	Lzz = 958.254-->
     <visual>
       <origin xyz="0 0 0" rpy="0 0 0" />
@@ -192,8 +237,8 @@
       <material name=""> <color rgba="1 1 1 1" /> </material>
     </visual>
-    <collision>
+    <!--collision>
       <origin xyz="0 0 0" rpy="0 0 0" />
       <geometry> <mesh filename="package://robot_description/meshes/Link_1.STL" /> </geometry>
-    </collision>
+    </collision-->
   </link>
   <joint name="Joint${number}_1" type="revolute">
@@ -215,4 +260,6 @@
       <inertia ixx="0.000909959" ixy="0" ixz="0.000569994" iyy="0.018834040" iyz="0" izz="0.018336908" />
     </inertial>
+<!--重心:(毫米)	X = 273.270	Y = 0.006	Z = 7.530
+    惯性张量:(千克*平方毫米)由重心决定，并且对齐输出的坐标系。Lxx = 909.959	Lxy = 0.824	Lxz = 569.994	Lyy = 18834.040	Lyz = 0.056	Lzz = 18336.908-->
     <visual>
       <origin xyz="0 0 0" rpy="0 0 0" />
@@ -221,6 +268,7 @@
     </visual>
     <collision>
-      <origin xyz="0 0 0" rpy="0 0 0" />
-      <geometry> <mesh filename="package://robot_description/meshes/Link_2.STL" /> </geometry>
+      <origin xyz="0.155 0 0" rpy="0 ${pi/2} 0" />
+      <geometry><cylinder length="0.3" radius="0.02" /></geometry>
+      <!--geometry> <mesh filename="package://robot_description/meshes/Link_2.STL" /> </geometry-->
     </collision>
   </link>
@@ -243,4 +291,6 @@
       <inertia ixx="0.000576423" ixy="0" ixz="0.000031283" iyy="0.001662107" iyz="0" izz="0.001334389" />
     </inertial>
+<!--重心:(毫米)	X = 81.336 Y = -0.003	Z = -0.693
+    惯性张量:(千克*平方毫米)由重心决定，并且对齐输出的坐标系。Lxx = 576.423	Lxy = -0.053 Lxz = 31.283 Lyy = 1662.107	Lyz = -0.009 Lzz = 1334.389-->
     <visual>
       <origin xyz="0 0 0" rpy="0 0 0" />
@@ -249,6 +299,7 @@
     </visual>
     <collision>
-      <origin xyz="0 0 0" rpy="0 0 0" />
-      <geometry> <mesh filename="package://robot_description/meshes/Link_3.STL" /> </geometry>
+      <origin xyz="0.16 0 0" rpy="0 ${pi/2} 0" />
+      <geometry><cylinder length="0.2" radius="0.02" /></geometry>
+      <!--geometry> <mesh filename="package://robot_description/meshes/Link_3.STL" /> </geometry-->
     </collision>
   </link>
@@ -271,4 +322,6 @@
       <inertia ixx="0.0001484574" ixy="0" ixz="0.000099045" iyy="0.001658464" iyz="-0.000002871" izz="0.000360737" />
     </inertial>
+<!--重心:(毫米)	X = 5.438	Y = 0.120	Z = 134.002
+    惯性张量:(千克*平方毫米)由重心决定，并且对齐输出的坐标系。Lxx = 1484.574	Lxy = -0.250 Lxz = 99.045 Lyy = 1658.464 Lyz = -2.871 Lzz = 360.737-->
     <visual>
       <origin xyz="0 0 0" rpy="0 0 0" />
@@ -276,8 +329,8 @@
       <material name=""> <color rgba="1 1 1 1" /> </material>
     </visual>
-    <collision>
-      <origin xyz="0 0 0" rpy="0 0 0" />
+    <!--collision>
+      <origin xyz="0 0 0.08" rpy="0 0 0" />
       <geometry> <mesh filename="package://robot_description/meshes/Link_4.STL" /> </geometry>
-    </collision>
+    </collision-->
   </link>
   <joint name="Joint${number}_4" type="revolute">
@@ -299,4 +352,6 @@
       <inertia ixx="0.000412080" ixy="0" ixz="0.000002889" iyy="0.000943104" iyz="0" izz="0.000708641" />
     </inertial>
+    <!--重心:(毫米)	X = 58.277 Y = 0.004 Z = -1.068
+        惯性张量:(千克*平方毫米)由重心决定，并且对齐输出的坐标系。Lxx = 412.080	Lxy = 0.032	Lxz = 2.889	Lyy = 943.104	Lyz = -0.003 Lzz = 708.641-->
     <visual>
       <origin xyz="0 0 0" rpy="0 0 0" />
@@ -304,8 +359,8 @@
       <material name=""> <color rgba="1 1 1 1" /> </material>
     </visual>
-    <collision>
-      <origin xyz="0 0 0" rpy="0 0 0" />
+    <!--collision>
+      <origin xyz="0.08 0 0" rpy="0 0 0" />
       <geometry> <mesh filename="package://robot_description/meshes/Link_5.STL" /> </geometry>
-    </collision>
+    </collision-->
   </link>
   <joint name="Joint${number}_5" type="revolute">
@@ -327,4 +382,6 @@
       <inertia ixx="0.000945510" ixy="-0.000011196" ixz="0" iyy="0.000811306" iyz="-0.000011704" izz="0.000402389" />
     </inertial>
+<!--重心:(毫米)	X = -0.094 Y = -1.809 Z = 70.443
+    惯性张量:(千克*平方毫米)由重心决定，并且对齐输出的坐标系。Lxx = 945.510	Lxy = -11.196	Lxz = -0.115	Lyy = 811.306	Lyz = -11.704	Lzz = 402.389-->
     <visual>
       <origin xyz="0 0 0" rpy="0 0 0" />
@@ -333,6 +390,7 @@
     </visual>
     <collision>
-      <origin xyz="0 0 0" rpy="0 0 0" />
-      <geometry> <mesh filename="package://robot_description/meshes/Link_6.STL" /> </geometry>
+      <origin xyz="0 0 -0.06" rpy="0 0 0" />
+      <geometry><cylinder length="0.1" radius="0.02" /></geometry>
+      <!--geometry> <mesh filename="package://robot_description/meshes/Link_6.STL" /> </geometry-->
     </collision>
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