Commit message: temp

File: src/robot_description/urdf/robot_description.urdf (robot description, URDF)
Before this commit: robot robot_description, 98 links, 97 joints
Links:
- removed link cube_l
- removed link cube_r
- removed link dummy_link
- removed link dummy_point1
- removed link dummy_point2
- removed link dummy_point3
- removed link dummy_point4
- removed link flan1
- removed link flan2
- removed link flan3
- removed link flan4
- removed link object
- removed link object1
- removed link object2
- link Link1_0: geometry collision mesh filename=package://robot_description/meshes/Link_0.STL; visual mesh filename=package://robot_description/meshes/Link_0.STL
- link Link1_1: geometry collision mesh filename=package://robot_description/meshes/Link_1.STL; visual mesh filename=package://robot_description/meshes/Link_1.STL
- link Link1_2: geometry collision mesh filename=package://robot_description/meshes/Link_2.STL; visual mesh filename=package://robot_description/meshes/Link_2.STL
- link Link1_3: geometry collision mesh filename=package://robot_description/meshes/Link_3.STL; visual mesh filename=package://robot_description/meshes/Link_3.STL
- link Link1_4: geometry collision mesh filename=package://robot_description/meshes/Link_4.STL; visual mesh filename=package://robot_description/meshes/Link_4.STL
- link Link1_5: geometry collision mesh filename=package://robot_description/meshes/Link_5.STL; visual mesh filename=package://robot_description/meshes/Link_5.STL
- link Link1_6: geometry collision mesh filename=package://robot_description/meshes/Link_6.STL; visual mesh filename=package://robot_description/meshes/Link_6.STL
- link Link1_platlink: geometry collision mesh filename=package://robot_description/meshes/Link_platlink.STL; visual mesh filename=package://robot_description/meshes/Link_platlink.STL
- link Link1_platlink2: geometry collision mesh filename=package://robot_description/meshes/Link_platlink2.STL; visual mesh filename=package://robot_description/meshes/Link_platlink2.STL
- link Link2_0: geometry collision mesh filename=package://robot_description/meshes/Link_0.STL; visual mesh filename=package://robot_description/meshes/Link_0.STL
- link Link2_1: geometry collision mesh filename=package://robot_description/meshes/Link_1.STL; visual mesh filename=package://robot_description/meshes/Link_1.STL
- link Link2_2: geometry collision mesh filename=package://robot_description/meshes/Link_2.STL; visual mesh filename=package://robot_description/meshes/Link_2.STL
- link Link2_3: geometry collision mesh filename=package://robot_description/meshes/Link_3.STL; visual mesh filename=package://robot_description/meshes/Link_3.STL
- link Link2_4: geometry collision mesh filename=package://robot_description/meshes/Link_4.STL; visual mesh filename=package://robot_description/meshes/Link_4.STL
- link Link2_5: geometry collision mesh filename=package://robot_description/meshes/Link_5.STL; visual mesh filename=package://robot_description/meshes/Link_5.STL
- link Link2_6: geometry collision mesh filename=package://robot_description/meshes/Link_6.STL; visual mesh filename=package://robot_description/meshes/Link_6.STL
- link Link2_platlink: geometry collision mesh filename=package://robot_description/meshes/Link_platlink.STL; visual mesh filename=package://robot_description/meshes/Link_platlink.STL
- link Link2_platlink2: geometry collision mesh filename=package://robot_description/meshes/Link_platlink2.STL; visual mesh filename=package://robot_description/meshes/Link_platlink2.STL
- link Link3_0: geometry collision mesh filename=package://robot_description/meshes/Link_0.STL; visual mesh filename=package://robot_description/meshes/Link_0.STL
- link Link3_1: geometry collision mesh filename=package://robot_description/meshes/Link_1.STL; visual mesh filename=package://robot_description/meshes/Link_1.STL
- link Link3_2: geometry collision mesh filename=package://robot_description/meshes/Link_2.STL; visual mesh filename=package://robot_description/meshes/Link_2.STL
- link Link3_3: geometry collision mesh filename=package://robot_description/meshes/Link_3.STL; visual mesh filename=package://robot_description/meshes/Link_3.STL
- link Link3_4: geometry collision mesh filename=package://robot_description/meshes/Link_4.STL; visual mesh filename=package://robot_description/meshes/Link_4.STL
- link Link3_5: geometry collision mesh filename=package://robot_description/meshes/Link_5.STL; visual mesh filename=package://robot_description/meshes/Link_5.STL
- link Link3_6: geometry collision mesh filename=package://robot_description/meshes/Link_6.STL; visual mesh filename=package://robot_description/meshes/Link_6.STL
- link Link3_platlink: geometry collision mesh filename=package://robot_description/meshes/Link_platlink.STL; visual mesh filename=package://robot_description/meshes/Link_platlink.STL
- link Link3_platlink2: geometry collision mesh filename=package://robot_description/meshes/Link_platlink2.STL; visual mesh filename=package://robot_description/meshes/Link_platlink2.STL
- link Link4_0: geometry collision mesh filename=package://robot_description/meshes/Link_0.STL; visual mesh filename=package://robot_description/meshes/Link_0.STL
- link Link4_1: geometry collision mesh filename=package://robot_description/meshes/Link_1.STL; visual mesh filename=package://robot_description/meshes/Link_1.STL
- link Link4_2: geometry collision mesh filename=package://robot_description/meshes/Link_2.STL; visual mesh filename=package://robot_description/meshes/Link_2.STL
- link Link4_3: geometry collision mesh filename=package://robot_description/meshes/Link_3.STL; visual mesh filename=package://robot_description/meshes/Link_3.STL
- link Link4_4: geometry collision mesh filename=package://robot_description/meshes/Link_4.STL; visual mesh filename=package://robot_description/meshes/Link_4.STL
- link Link4_5: geometry collision mesh filename=package://robot_description/meshes/Link_5.STL; visual mesh filename=package://robot_description/meshes/Link_5.STL
- link Link4_6: geometry collision mesh filename=package://robot_description/meshes/Link_6.STL; visual mesh filename=package://robot_description/meshes/Link_6.STL
- link Link4_platlink: geometry collision mesh filename=package://robot_description/meshes/Link_platlink.STL; visual mesh filename=package://robot_description/meshes/Link_platlink.STL
- link Link4_platlink2: geometry collision mesh filename=package://robot_description/meshes/Link_platlink2.STL; visual mesh filename=package://robot_description/meshes/Link_platlink2.STL
- link Link_platform: geometry collision mesh filename=package://robot_description/meshes/Link_platform.STL; visual mesh filename=package://robot_description/meshes/Link_platform.STL
- link base_link: geometry collision mesh filename=package://robot_description/meshes/base_link.STL; visual mesh filename=package://robot_description/meshes/base_link.STL
Joints:
- removed joint dummy_joint
- removed joint flan_joint1
- removed joint flan_joint2
- removed joint flan_joint3
- removed joint flan_joint4
- removed joint truss_link_to_cube_l
- removed joint truss_link_to_cube_r
- removed joint truss_link_to_obj
- removed joint truss_link_to_obj1
- removed joint truss_link_to_obj2
- removed joint truss_link_to_point1
- removed joint truss_link_to_point2
- removed joint truss_link_to_point3
- removed joint truss_link_to_point4
- joint world_joint: child dummy_link -> base_link
