Commit message: moveit更改

File: src/robot_description/urdf/robot_description.urdf (robot description, URDF)
Before this commit: robot robot_description, 84 links, 83 joints
Links:
- removed link Link1_platlink2
- removed link Link2_platlink2
- removed link Link3_platlink2
- removed link Link4_platlink2
- added link cube_l
- added link cube_r
- added link dummy_point1
- added link dummy_point2
- added link dummy_point3
- added link dummy_point4
- added link object
- added link object1
- added link object2
Joints:
- removed joint Joint1_platlink2
- removed joint Joint2_platlink2
- removed joint Joint3_platlink2
- removed joint Joint4_platlink2
- added joint truss_link_to_cube_l: type fixed, parent truss_link, child cube_l, origin xyz=-0.1175 0.12 0.2325 rpy=0 3.1416 0
- added joint truss_link_to_cube_r: type fixed, parent truss_link, child cube_r, origin xyz=-0.1175 0.12 -0.2325 rpy=0 0 0
- added joint truss_link_to_obj: type fixed, parent truss_link, child object, origin xyz=0.08 0.03 0.40 rpy=1.5708 0.707 0
- added joint truss_link_to_obj1: type fixed, parent truss_link, child object1, origin xyz=-0.1 0.215 0.085 rpy=0 3.1416 0
- added joint truss_link_to_obj2: type fixed, parent truss_link, child object2, origin xyz=-0.265 0.215 -0.35 rpy=0 0 -1.5708
- added joint truss_link_to_point1: type fixed, parent truss_link, child dummy_point1, origin xyz=0.795 0 0.53 rpy=1.5708 0 0
- added joint truss_link_to_point2: type fixed, parent truss_link, child dummy_point2, origin xyz=0.795 0 -0.53 rpy=1.5708 0 0
- added joint truss_link_to_point3: type fixed, parent truss_link, child dummy_point3, origin xyz=0.08 0.18 0.40 rpy=1.5708 0.707 0
- added joint truss_link_to_point4: type fixed, parent truss_link, child dummy_point4, origin xyz=0 0.215 -0.3 rpy=0 0 0

File: src/robot_description/urdf/robot_description.xacro (robot description, xacro)
@@ -73,5 +73,5 @@
     </collision>
   </link>
-  <!-- <link name="dummy_point1"></link>
+  <link name="dummy_point1"></link>
   <joint name="truss_link_to_point1" type="fixed">
     <parent link="truss_link"/>
@@ -126,5 +126,5 @@
     <child link="cube_r"/>
     <origin xyz="-0.1175 0.12 -0.2325" rpy="0 0 0"/>
-  </joint> -->
+  </joint>
   <link name="Link_platform">
     <inertial>
@@ -385,31 +385,4 @@
     <limit
       lower="${-pi/2}"
-      upper="0"
-      effort="1000"
-      velocity="10" />
-  </joint>
-  <link name="Link${number}_platlink2">
-    <inertial>
-      <origin xyz="-0.033084 0.0135522 0.00049999" rpy="0 0 0" />
-      <mass value="0.0110" />
-      <inertia ixx="2.3755012E-06" ixy="4.9413420E-06" ixz="0" iyy="1.2414435E-05" iyz="0" izz="1.4621084E-05" />
-    </inertial>
-    <visual>
-      <origin xyz="0 0 0" rpy="0 0 0" />
-      <geometry> <mesh filename="package://robot_description/meshes/Link_platlink2.STL" /> </geometry>
-      <material name=""> <color rgba="1 1 1 1" /> </material>
-    </visual>
-    <collision>
-      <origin xyz="0 0 0" rpy="0 0 0" />
-      <geometry> <mesh filename="package://robot_description/meshes/Link_platlink2.STL" /> </geometry>
-    </collision>
-  </link>
-  <joint name="Joint${number}_platlink2" type="revolute">
-    <origin xyz="0.04 0 0" rpy="0 0 0" />
-    <parent link="Link${number}_0" />
-    <child link="Link${number}_platlink2" />
-    <axis xyz="0 0 1" />
-    <limit
-      lower="-${pi/2}"
       upper="0"
       effort="1000"

Commit message: moveit修复base_link固定bug

File: src/robot_description/urdf/robot_description.urdf (robot description, URDF)
Before this commit: robot robot_description, 89 links, 88 joints
Links:
- removed link cube_l
- removed link cube_r
- removed link dummy_point1
- removed link dummy_point2
- removed link dummy_point3
- removed link dummy_point4
- removed link object
- removed link object1
- removed link object2
- removed link truss_link
- removed link world
- link Link1_left_inner_finger_pad: mass None -> 0.1
- link Link1_right_inner_finger_pad: mass None -> 0.1
- link Link2_left_inner_finger_pad: mass None -> 0.1
- link Link2_right_inner_finger_pad: mass None -> 0.1
- link Link3_left_inner_finger_pad: mass None -> 0.1
- link Link3_right_inner_finger_pad: mass None -> 0.1
- link Link4_left_inner_finger_pad: mass None -> 0.1
- link Link4_right_inner_finger_pad: mass None -> 0.1
Joints:
- removed joint truss_link_to_cube_l
- removed joint truss_link_to_cube_r
- removed joint truss_link_to_obj
- removed joint truss_link_to_obj1
- removed joint truss_link_to_obj2
- removed joint truss_link_to_point1
- removed joint truss_link_to_point2
- removed joint truss_link_to_point3
- removed joint truss_link_to_point4
- removed joint world_joint
- removed joint world_to_truss_link

File: src/robot_description/urdf/robot_description.xacro (robot description, xacro)
@@ -11,34 +11,13 @@
   <joint name="world_joint" type="fixed">
     <parent link="world"/>
-    <child  link="base_link"/>
+    <child  link="dummy_link"/>
     <origin xyz="0 0 0.45" rpy="0 1.5708 0"/>
   </joint>
-  <link name="base_link">
-    <inertial>
-      <origin xyz="0 0 0.042" rpy="0 0 0" />
-      <mass value="1.492" />
-      <inertia ixx="0.004886486" ixy="-0.000017397" ixz="-0.000263075" iyy="0.004100237" iyz="0" izz="0.003937989" />
-    </inertial>
-    <visual>
-      <origin xyz="0 0 0" rpy="0 0 0" />
-      <geometry> <mesh filename="package://robot_description/meshes/base_link.STL" /> </geometry>
-      <material name=""> <color rgba="0.75294 0.75294 0.75294 1" /> </material>
-    </visual>
-    <collision>
-      <origin xyz="0 0 0" rpy="0 0 0" />
-      <geometry>
-        <mesh filename="package://robot_description/meshes/base_link.STL"/>
-      </geometry>
-      <surface>
-        <friction>
-          <torsional>
-            <coefficient>5.0</coefficient>
-            <surface_radius>0.10</surface_radius>
-            <use_patch_radius>false</use_patch_radius>
-          </torsional>
-        </friction>
-      </surface>
-    </collision>
-  </link>
+  <link name="dummy_link"></link>
+  <joint name="dummy_joint" type="fixed">
+      <parent link="dummy_link"/>
+      <child  link="base_link"/>
+      <origin xyz="0 0 0" rpy="0 0 0"/>
+  </joint>
   <joint name="world_to_truss_link" type="fixed">
     <parent link="world"/>

Commit message: temp

File: src/robot_description/urdf/robot_description.urdf (robot description, URDF)
Before this commit: robot robot_description, 78 links, 77 joints
Links:
- added link dummy_root
Joints:
- added joint dummy_fixed_joint: type fixed, parent dummy_root, child base_link, origin xyz=0 0 0 rpy=0 0 0
