Commit message: 注释Link${number}_platlink2相关

File: src/robot_description/urdf/robot_description_copy.xacro (robot description, xacro)
@@ -478,5 +478,5 @@
       velocity="10" />
   </joint>
-    <link
+  <!-- <link
     name="Link${number}_platlink2">
     <inertial>
@@ -489,23 +489,23 @@
       <geometry> <mesh filename="package://robot_description/meshes/Link_platlink2.STL" /> </geometry>
       <material name=""> <color rgba="1 1 1 1" /> </material>
-    </visual>
+    </visual> -->
     <!--collision>
       <origin xyz="0 0 0" rpy="0 0 0" />
       <geometry> <mesh filename="package://robot_description/meshes/Link_platlink2.STL" /> </geometry>
     </collision-->
-  </link>
-  <joint name="Joint${number}_platlink2" type="revolute">
-    <origin xyz="0.04 0 0" rpy="0 0 0" />
-    <parent link="Link${number}_0" />
-    <child link="Link${number}_platlink2" />
-    <axis xyz="0 0 1" />
+  <!-- </link> -->
+  <!-- <joint name="Joint${number}_platlink2" type="revolute"> -->
+    <!-- <origin xyz="0.04 0 0" rpy="0 0 0" /> -->
+    <!-- <parent link="Link${number}_0" /> -->
+    <!-- <child link="Link${number}_platlink2" /> -->
+    <!-- <axis xyz="0 0 1" /> -->
     <!--xacro:insert_block name="dynamics_parameter"/-->
-    <limit
+    <!-- <limit
       lower="-${pi/2}"
       upper="0"
       effort="1000"
-      velocity="10" />
-  </joint>
-    <gazebo>
+      velocity="10" /> -->
+  <!-- </joint> -->
+  <!-- <gazebo>
     <joint name="joint${number}_connect" type="fixed">
       <pose>0 0 0 0 0 0</pose>
@@ -513,5 +513,5 @@
       <child>Link${number}_platlink2</child>
     </joint>
-  </gazebo>
+  </gazebo> -->
 </xacro:macro>
 <!--ALL Leg Set*******************************************************************************************-->

Commit message: temp

File: src/robot_description/urdf/robot_description_copy.xacro (robot description, xacro)
@@ -83,5 +83,5 @@
     <child link="dummy_point3"/>
     <!-- 如果需要在 truss_link 坐标系中给 base_link 设置一个平移或姿态偏移，可以在这里修改 xyz / rpy -->
-    <origin xyz="0.08 0.18 0.40" rpy="1.5708 0.707 0"/>
+    <origin xyz="0.08 0.23 0.36" rpy="1.5708 1.047 0"/>
   </joint>
   <link name="dummy_point3"></link>
@@ -99,5 +99,5 @@
     <!-- 如果需要在 truss_link 坐标系中给 base_link 设置一个平移或姿态偏移，可以在这里修改 xyz / rpy -->
     <!-- 转换到joint2_6______0.1 -->
-    <origin xyz="0.08 0.03 0.40" rpy="1.5708 0.707 0"/>
+    <origin xyz="0.08 0.0 0.36" rpy="1.5708 1.047 0"/>
   </joint>
   <link name="object"></link>

Commit message: 相机

File: src/robot_description/urdf/robot_description_copy.xacro (robot description, xacro)
@@ -19,4 +19,10 @@
       <child  link="base_link"/>
       <origin xyz="0 0 0" rpy="0 0 0"/>
+  </joint>
+  <link name="camera_link"/>
+  <joint name="camera_joint" type="fixed">
+      <parent link="base_link"/>
+      <child link="camera_link"/>
+      <origin xyz="0.1 0.05 0.2" rpy="-0.7071 0 -1.5708"/>
   </joint>
   <joint name="world_to_truss_link" type="fixed">

Commit message: temp

File: src/robot_description/urdf/robot_description_copy.xacro (robot description, xacro)
@@ -89,5 +89,5 @@
     <child link="dummy_point3"/>
     <!-- 如果需要在 truss_link 坐标系中给 base_link 设置一个平移或姿态偏移，可以在这里修改 xyz / rpy -->
-    <origin xyz="0.08 0.23 0.36" rpy="1.5708 1.047 0"/>
+    <origin xyz="0.08 0.13 0.36" rpy="1.5708 1.047 0"/>
   </joint>
   <link name="dummy_point3"></link>

Commit message: 相机位姿

File: src/robot_description/urdf/robot_description_copy.xacro (robot description, xacro)
@@ -24,5 +24,5 @@
       <parent link="base_link"/>
       <child link="camera_link"/>
-      <origin xyz="0.1 0.05 0.2" rpy="-0.7071 0 -1.5708"/>
+      <origin xyz="0.16893 0.0325 0.11643" rpy="-0.7071 0 -1.5708"/>
   </joint>
   <joint name="world_to_truss_link" type="fixed">

Commit message: temp

File: src/robot_description/urdf/robot_description_copy.xacro (robot description, xacro)
@@ -113,5 +113,5 @@
     <!-- 如果需要在 truss_link 坐标系中给 base_link 设置一个平移或姿态偏移，可以在这里修改 xyz / rpy -->
     <!-- 转换到joint2_6______0.1 -->
-    <origin xyz="-0.1 0.215 0.085" rpy="0 3.1416 0"/>
+    <origin xyz="-0.1 0.215 0.085" rpy="0 3.1416 -3.1416"/>
   </joint>
   <link name="object1"></link>
@@ -131,4 +131,12 @@
     <!-- 转换到joint2_6______0.1 -->
     <origin xyz="-0.1175 0.12 0.2325" rpy="0 3.1416 0"/>
+  </joint>
+  <link name="cube_m"></link>
+  <joint name="truss_link_to_cube_m" type="fixed">
+    <parent link="truss_link"/>
+    <child link="cube_m"/>
+    <!-- 如果需要在 truss_link 坐标系中给 base_link 设置一个平移或姿态偏移，可以在这里修改 xyz / rpy -->
+    <!-- 转换到joint2_6______0.1 -->
+    <origin xyz="-0.1175 0.12 0" rpy="0 0 0"/>
   </joint>
   <link name="cube_r"></link>

Commit message: temp

File: src/robot_description/urdf/robot_description_copy.xacro (robot description, xacro)
@@ -130,5 +130,5 @@
     <!-- 如果需要在 truss_link 坐标系中给 base_link 设置一个平移或姿态偏移，可以在这里修改 xyz / rpy -->
     <!-- 转换到joint2_6______0.1 -->
-    <origin xyz="-0.1175 0.12 0.2325" rpy="0 3.1416 0"/>
+    <origin xyz="-0.1175 0.12 0.2325" rpy="0 3.1416 3.1416"/>
   </joint>
   <link name="cube_m"></link>

Commit message: temp

File: src/robot_description/urdf/robot_description_copy.xacro (robot description, xacro)
@@ -130,5 +130,5 @@
     <!-- 如果需要在 truss_link 坐标系中给 base_link 设置一个平移或姿态偏移，可以在这里修改 xyz / rpy -->
     <!-- 转换到joint2_6______0.1 -->
-    <origin xyz="-0.1175 0.12 0.2325" rpy="0 3.1416 3.1416"/>
+    <origin xyz="-0.1175 0.15 0.1725" rpy="0 3.1416 3.1416"/>
   </joint>
   <link name="cube_m"></link>
@@ -138,5 +138,5 @@
     <!-- 如果需要在 truss_link 坐标系中给 base_link 设置一个平移或姿态偏移，可以在这里修改 xyz / rpy -->
     <!-- 转换到joint2_6______0.1 -->
-    <origin xyz="-0.1175 0.12 0" rpy="0 0 0"/>
+    <origin xyz="-0.1175 0.15 0" rpy="0 0 0"/>
   </joint>
   <link name="cube_r"></link>
@@ -146,5 +146,5 @@
     <!-- 如果需要在 truss_link 坐标系中给 base_link 设置一个平移或姿态偏移，可以在这里修改 xyz / rpy -->
     <!-- 转换到joint2_6______0.1 -->
-    <origin xyz="-0.1175 0.12 -0.2325" rpy="0 0 0"/>
+    <origin xyz="-0.1175 0.15 -0.1725" rpy="0 0 0"/>
   </joint>
   <link name="base_link">

Commit message: temp

File: src/robot_description/urdf/robot_description_copy.xacro (robot description, xacro)
@@ -121,5 +121,5 @@
     <!-- 如果需要在 truss_link 坐标系中给 base_link 设置一个平移或姿态偏移，可以在这里修改 xyz / rpy -->
     <!-- 转换到joint2_6______0.1 -->
-    <origin xyz="-0.265 0.215 -0.35" rpy="0 0 -1.5708"/>
+    <origin xyz="-0.265 0.215 -0.35" rpy="0 0 1.5708"/>
   </joint>
   <link name="object2"></link>

Commit message: temp

File: src/robot_description/urdf/robot_description_copy.xacro (robot description, xacro)
@@ -147,4 +147,87 @@
     <!-- 转换到joint2_6______0.1 -->
     <origin xyz="-0.1175 0.15 -0.1725" rpy="0 0 0"/>
+  </joint>
+  <!-- <link name="grasp_object_cube">
+    <inertial>
+      <origin
+        xyz="0.132500000000003 0.132499999999999 -0.0662499999999996"
+        rpy="0 0 0" />
+      <mass
+        value="1.47124857062568" />
+      <inertia
+        ixx="0.0232365321123193"
+        ixy="-7.32404384667322E-17"
+        ixz="2.07830204072989E-16"
+        iyy="0.0232365321123194"
+        iyz="1.96889159156655E-16"
+        izz="0.0387444115770706" />
+    </inertial>
+    <visual>
+      <origin
+        xyz="0 0 0"
+        rpy="0 0 0" />
+      <geometry>
+        <mesh
+          filename="package://object_cube/meshes/base_link.STL" />
+      </geometry>
+      <material
+        name="">
+        <color
+          rgba="0.898039215686275 0.917647058823529 0.929411764705882 1" />
+      </material>
+    </visual>
+    <collision>
+      <origin
+        xyz="0 0 0"
+        rpy="0 0 0" />
+      <geometry>
+        <mesh
+          filename="package://object_cube/meshes/base_link.STL" />
+      </geometry>
+    </collision>
+  </link> -->
+  <link name="grasp_object">
+    <inertial>
+      <origin
+        xyz="-1.7465753580787E-17 1.31917654026282E-17 0.1"
+        rpy="0 0 0" />
+      <mass
+        value="0.156515805385711" />
+      <inertia
+        ixx="0"
+        ixy="0"
+        ixz="0"
+        iyy="0"
+        iyz="0"
+        izz="0" />
+    </inertial>
+    <visual>
+      <origin
+        xyz="0 0 0"
+        rpy="0 0 0" />
+      <geometry>
+        <mesh
+          filename="package://object/meshes/grasp_object.STL" />
+      </geometry>
+      <material
+        name="">
+        <color
+          rgba="0.898039215686275 0.917647058823529 0.929411764705882 1" />
+      </material>
+    </visual>
+    <collision>
+      <origin
+        xyz="0 0 0"
+        rpy="0 0 0" />
+      <geometry>
+        <mesh
+          filename="package://object/meshes/grasp_object.STL" />
+      </geometry>
+    </collision>
+  </link>
+  <joint name="world_to_grasp_object" type="fixed">
+    <parent link="world"/>
+    <child link="grasp_object"/>
+    <origin xyz="0.59 0.373 -0.07" rpy="0 0 0"/>
   </joint>
   <link name="base_link">

Commit message: temp

File: src/robot_description/urdf/robot_description_copy.xacro (robot description, xacro)
@@ -187,5 +187,5 @@
     </collision>
   </link> -->
-  <link name="grasp_object">
+  <!-- <link name="grasp_object">
     <inertial>
       <origin
@@ -230,4 +230,49 @@
     <child link="grasp_object"/>
     <origin xyz="0.59 0.373 -0.07" rpy="0 0 0"/>
+  </joint> -->
+  <link
+    name="grasp_object_cube">
+    <inertial>
+      <origin
+        xyz="0.132500000000003 0.132499999999999 -0.0662499999999996"
+        rpy="0 0 0" />
+      <mass
+        value="1.47124857062568" />
+      <inertia
+        ixx="0.0232365321123193"
+        ixy="-7.32404384667322E-17"
+        ixz="2.07830204072989E-16"
+        iyy="0.0232365321123194"
+        iyz="1.96889159156655E-16"
+        izz="0.0387444115770706" />
+    </inertial>
+    <visual>
+      <origin
+        xyz="0 0 0"
+        rpy="0 0 0" />
+      <geometry>
+        <mesh
+          filename="package://object_cube/meshes/grasp_object_cube.STL" />
+      </geometry>
+      <material
+        name="">
+        <color
+          rgba="0.898039215686275 0.917647058823529 0.929411764705882 1" />
+      </material>
+    </visual>
+    <collision>
+      <origin
+        xyz="0 0 0"
+        rpy="0 0 0" />
+      <geometry>
+        <mesh
+          filename="package://object_cube/meshes/grasp_object_cube.STL" />
+      </geometry>
+    </collision>
+  </link>
+  <joint name="world_to_grasp_object_cube" type="fixed">
+    <parent link="world"/>
+    <child link="grasp_object_cube"/>
+    <origin xyz="0.6625 0.0 0.0" rpy="0 0 0"/>
   </joint>
   <link name="base_link">

Commit message: temp

File: src/robot_description/urdf/robot_description_copy.xacro (robot description, xacro)
@@ -130,5 +130,5 @@
     <!-- 如果需要在 truss_link 坐标系中给 base_link 设置一个平移或姿态偏移，可以在这里修改 xyz / rpy -->
     <!-- 转换到joint2_6______0.1 -->
-    <origin xyz="-0.1175 0.15 0.1725" rpy="0 3.1416 3.1416"/>
+    <origin xyz="-0.1475 0.135 0.20" rpy="0 3.1416 3.1416"/>
   </joint>
   <link name="cube_m"></link>
@@ -138,5 +138,5 @@
     <!-- 如果需要在 truss_link 坐标系中给 base_link 设置一个平移或姿态偏移，可以在这里修改 xyz / rpy -->
     <!-- 转换到joint2_6______0.1 -->
-    <origin xyz="-0.1175 0.15 0" rpy="0 0 0"/>
+    <origin xyz="-0.1475 0.135 0" rpy="0 0 0"/>
   </joint>
   <link name="cube_r"></link>
@@ -146,5 +146,5 @@
     <!-- 如果需要在 truss_link 坐标系中给 base_link 设置一个平移或姿态偏移，可以在这里修改 xyz / rpy -->
     <!-- 转换到joint2_6______0.1 -->
-    <origin xyz="-0.1175 0.15 -0.1725" rpy="0 0 0"/>
+    <origin xyz="-0.1475 0.135 -0.20" rpy="0 0 0"/>
   </joint>
   <!-- <link name="grasp_object_cube">
@@ -274,5 +274,5 @@
     <parent link="world"/>
     <child link="grasp_object_cube"/>
-    <origin xyz="0.6625 0.0 0.0" rpy="0 0 0"/>
+    <origin xyz="0.6925 -0.1325 0.15" rpy="0 0 0"/>
   </joint>
   <link name="base_link">

Commit message: temp

File: src/robot_description/urdf/robot_description_copy.xacro (robot description, xacro)
@@ -132,4 +132,12 @@
     <origin xyz="-0.1475 0.135 0.20" rpy="0 3.1416 3.1416"/>
   </joint>
+  <link name="cube_l_pre"></link>
+  <joint name="truss_link_to_cube_l_pre" type="fixed">
+    <parent link="truss_link"/>
+    <child link="cube_l_pre"/>
+    <!-- 如果需要在 truss_link 坐标系中给 base_link 设置一个平移或姿态偏移，可以在这里修改 xyz / rpy -->
+    <!-- 转换到joint2_6______0.1 -->
+    <origin xyz="-0.1475 0.135 0.25" rpy="0 3.1416 3.1416"/>
+  </joint>
   <link name="cube_m"></link>
   <joint name="truss_link_to_cube_m" type="fixed">
@@ -147,4 +155,12 @@
     <!-- 转换到joint2_6______0.1 -->
     <origin xyz="-0.1475 0.135 -0.20" rpy="0 0 0"/>
+  </joint>
+  <link name="cube_r_pre"></link>
+  <joint name="truss_link_to_cube_r_pre" type="fixed">
+    <parent link="truss_link"/>
+    <child link="cube_r_pre"/>
+    <!-- 如果需要在 truss_link 坐标系中给 base_link 设置一个平移或姿态偏移，可以在这里修改 xyz / rpy -->
+    <!-- 转换到joint2_6______0.1 -->
+    <origin xyz="-0.1475 0.135 -0.25" rpy="0 0 0"/>
   </joint>
   <!-- <link name="grasp_object_cube">

Commit message: temp

File: src/robot_description/urdf/robot_description_copy.xacro (robot description, xacro)
@@ -130,5 +130,5 @@
     <!-- 如果需要在 truss_link 坐标系中给 base_link 设置一个平移或姿态偏移，可以在这里修改 xyz / rpy -->
     <!-- 转换到joint2_6______0.1 -->
-    <origin xyz="-0.1475 0.135 0.20" rpy="0 3.1416 3.1416"/>
+    <origin xyz="-0.1475 0.135 0.22" rpy="0 3.1416 3.1416"/>
   </joint>
   <link name="cube_l_pre"></link>
@@ -138,5 +138,5 @@
     <!-- 如果需要在 truss_link 坐标系中给 base_link 设置一个平移或姿态偏移，可以在这里修改 xyz / rpy -->
     <!-- 转换到joint2_6______0.1 -->
-    <origin xyz="-0.1475 0.135 0.25" rpy="0 3.1416 3.1416"/>
+    <origin xyz="-0.1475 0.135 0.35" rpy="0 3.1416 3.1416"/>
   </joint>
   <link name="cube_m"></link>
@@ -154,5 +154,5 @@
     <!-- 如果需要在 truss_link 坐标系中给 base_link 设置一个平移或姿态偏移，可以在这里修改 xyz / rpy -->
     <!-- 转换到joint2_6______0.1 -->
-    <origin xyz="-0.1475 0.135 -0.20" rpy="0 0 0"/>
+    <origin xyz="-0.1475 0.135 -0.22" rpy="0 0 0"/>
   </joint>
   <link name="cube_r_pre"></link>
@@ -162,5 +162,5 @@
     <!-- 如果需要在 truss_link 坐标系中给 base_link 设置一个平移或姿态偏移，可以在这里修改 xyz / rpy -->
     <!-- 转换到joint2_6______0.1 -->
-    <origin xyz="-0.1475 0.135 -0.25" rpy="0 0 0"/>
+    <origin xyz="-0.1475 0.135 -0.35" rpy="0 0 0"/>
   </joint>
   <!-- <link name="grasp_object_cube">

Commit message: temp

File: src/robot_description/urdf/robot_description_copy.xacro (robot description, xacro)
@@ -130,5 +130,13 @@
     <!-- 如果需要在 truss_link 坐标系中给 base_link 设置一个平移或姿态偏移，可以在这里修改 xyz / rpy -->
     <!-- 转换到joint2_6______0.1 -->
-    <origin xyz="-0.1475 0.135 0.20" rpy="0 3.1416 3.1416"/>
+    <origin xyz="-0.1475 0.135 0.22" rpy="0 3.1416 3.1416"/>
+  </joint>
+  <link name="cube_l_pre"></link>
+  <joint name="truss_link_to_cube_l_pre" type="fixed">
+    <parent link="truss_link"/>
+    <child link="cube_l_pre"/>
+    <!-- 如果需要在 truss_link 坐标系中给 base_link 设置一个平移或姿态偏移，可以在这里修改 xyz / rpy -->
+    <!-- 转换到joint2_6______0.1 -->
+    <origin xyz="-0.1475 0.135 0.35" rpy="0 3.1416 3.1416"/>
   </joint>
   <link name="cube_m"></link>
@@ -146,5 +154,13 @@
     <!-- 如果需要在 truss_link 坐标系中给 base_link 设置一个平移或姿态偏移，可以在这里修改 xyz / rpy -->
     <!-- 转换到joint2_6______0.1 -->
-    <origin xyz="-0.1475 0.135 -0.20" rpy="0 0 0"/>
+    <origin xyz="-0.1475 0.135 -0.22" rpy="0 0 0"/>
+  </joint>
+  <link name="cube_r_pre"></link>
+  <joint name="truss_link_to_cube_r_pre" type="fixed">
+    <parent link="truss_link"/>
+    <child link="cube_r_pre"/>
+    <!-- 如果需要在 truss_link 坐标系中给 base_link 设置一个平移或姿态偏移，可以在这里修改 xyz / rpy -->
+    <!-- 转换到joint2_6______0.1 -->
+    <origin xyz="-0.1475 0.135 -0.35" rpy="0 0 0"/>
   </joint>
   <!-- <link name="grasp_object_cube">

Commit message: temp

File: src/robot_description/urdf/robot_description_copy.xacro (robot description, xacro)
@@ -247,5 +247,5 @@
     <origin xyz="0.59 0.373 -0.07" rpy="0 0 0"/>
   </joint> -->
-  <link
+  <!-- <link
     name="grasp_object_cube">
     <inertial>
@@ -291,5 +291,5 @@
     <child link="grasp_object_cube"/>
     <origin xyz="0.6925 -0.1325 0.15" rpy="0 0 0"/>
-  </joint>
+  </joint> -->
   <link name="base_link">
     <inertial>

Commit message: temp

File: src/robot_description/urdf/robot_description_copy.xacro (robot description, xacro)
@@ -203,5 +203,5 @@
     </collision>
   </link> -->
-  <!-- <link name="grasp_object">
+  <link name="grasp_object">
     <inertial>
       <origin
@@ -245,6 +245,6 @@
     <parent link="world"/>
     <child link="grasp_object"/>
-    <origin xyz="0.59 0.373 -0.07" rpy="0 0 0"/>
-  </joint> -->
+    <origin xyz="0.59 0.373 -0.07" rpy="0 0 -0.5238"/>
+  </joint>
   <!-- <link
     name="grasp_object_cube">

Commit message: temp

File: src/robot_description/urdf/robot_description_copy.xacro (robot description, xacro)
@@ -130,5 +130,5 @@
     <!-- 如果需要在 truss_link 坐标系中给 base_link 设置一个平移或姿态偏移，可以在这里修改 xyz / rpy -->
     <!-- 转换到joint2_6______0.1 -->
-    <origin xyz="-0.1475 0.135 0.22" rpy="0 3.1416 3.1416"/>
+    <origin xyz="-0.1175 0.235 0.22" rpy="0 3.1416 3.1416"/>
   </joint>
   <link name="cube_l_pre"></link>
@@ -138,5 +138,5 @@
     <!-- 如果需要在 truss_link 坐标系中给 base_link 设置一个平移或姿态偏移，可以在这里修改 xyz / rpy -->
     <!-- 转换到joint2_6______0.1 -->
-    <origin xyz="-0.1475 0.135 0.35" rpy="0 3.1416 3.1416"/>
+    <origin xyz="-0.1175 0.235 0.35" rpy="0 3.1416 3.1416"/>
   </joint>
   <link name="cube_m"></link>
@@ -146,5 +146,5 @@
     <!-- 如果需要在 truss_link 坐标系中给 base_link 设置一个平移或姿态偏移，可以在这里修改 xyz / rpy -->
     <!-- 转换到joint2_6______0.1 -->
-    <origin xyz="-0.1475 0.135 0" rpy="0 0 0"/>
+    <origin xyz="-0.1175 0.235 0" rpy="0 0 0"/>
   </joint>
   <link name="cube_r"></link>
@@ -154,5 +154,5 @@
     <!-- 如果需要在 truss_link 坐标系中给 base_link 设置一个平移或姿态偏移，可以在这里修改 xyz / rpy -->
     <!-- 转换到joint2_6______0.1 -->
-    <origin xyz="-0.1475 0.135 -0.22" rpy="0 0 0"/>
+    <origin xyz="-0.1175 0.235 -0.22" rpy="0 0 0"/>
   </joint>
   <link name="cube_r_pre"></link>
@@ -162,5 +162,5 @@
     <!-- 如果需要在 truss_link 坐标系中给 base_link 设置一个平移或姿态偏移，可以在这里修改 xyz / rpy -->
     <!-- 转换到joint2_6______0.1 -->
-    <origin xyz="-0.1475 0.135 -0.35" rpy="0 0 0"/>
+    <origin xyz="-0.1175 0.235 -0.35" rpy="0 0 0"/>
   </joint>
   <!-- <link name="grasp_object_cube">
@@ -290,5 +290,5 @@
     <parent link="world"/>
     <child link="grasp_object_cube"/>
-    <origin xyz="0.6925 -0.1325 0.15" rpy="0 0 0"/>
+    <origin xyz="0.6625 -0.1325 0.25" rpy="0 0 0"/>
   </joint>
   <link name="base_link">
